Commit message: driveable robot for 2_wheel template

File: simulation_ws/src/two_wheel_robot/urdf/4_two_wheel_robot.xacro (robot description, xacro)
@@ -67,5 +67,4 @@
       <origin rpy="0 0 0" xyz="0 0 0"/>
       <geometry>
-        <!-- <box size="0.5 0.3 0.07"/> -->
         <box size="1.0 0.6 0.07"/>
       </geometry>
@@ -90,5 +89,4 @@
     </collision>
     <visual name="caster_front_visual">
-      <!-- <origin rpy=" 0 0 0" xyz="0.2 0 -0.05"/> -->
       <origin rpy=" 0 0 0" xyz="0.2 0 -0.03"/>
       <geometry>
@@ -96,13 +94,36 @@
       </geometry>
     </visual>
+    <!-- caster rear -->
+    <collision name="caster_front_collision">
+    <origin rpy=" 0 0 0" xyz="-0.35 0 -0.05"/>
+      <geometry>
+        <sphere radius="0.05"/>
+      </geometry>
+      <surface>
+        <friction>
+          <ode>
+            <mu>0</mu>
+            <mu2>0</mu2>
+            <slip1>1.0</slip1>
+            <slip2>1.0</slip2>
+          </ode>
+        </friction>
+      </surface>
+    </collision>
+    <visual name="caster_front_visual">
+      <origin rpy=" 0 0 0" xyz="-0.2 0 -0.03"/>
+      <geometry>
+        <sphere radius="0.05"/>
+      </geometry>
+    </visual>
   </link>
   <link name="link_right_wheel">
     <inertial>
       <mass value="0.2"/>
-      <origin rpy="0 1.5707 1.5707" xyz="0 0 0"/>
+      <origin rpy="0 1.5707 1.5707" xyz="0.15 0.15 0"/>
       <inertia ixx="0.000526666666667" ixy="0" ixz="0" iyy="0.000526666666667" iyz="0" izz="0.001"/>
     </inertial>
     <collision name="link_right_wheel_collision">
-      <origin rpy="0 1.5707 1.5707" xyz="0 0 0"/>
+      <origin rpy="0 1.5707 1.5707" xyz="-0.15 0.15 0"/>
       <geometry>
         <cylinder length="0.04" radius="0.1"/>
@@ -110,14 +131,12 @@
     </collision>
     <visual name="link_right_wheel_visual">
-      <!-- <origin rpy="0 1.5707 1.5707" xyz="0 0 0"/> -->
-      <origin rpy="0 1.5707 1.5707" xyz="-0.1 0.15 0"/>
-      <geometry>
-        <cylinder length="0.06" radius="0.1"/>
-        <!-- <cylinder length="0.04" radius="0.1"/> -->
+      <origin rpy="0 1.5707 1.5707" xyz="-0.15 0.15 0"/>
+      <geometry>
+        <cylinder length="0.06" radius="0.1"/>
       </geometry>
     </visual>
   </link>
   <joint name="joint_right_wheel" type="continuous">
-    <origin rpy="0 0 0" xyz="-0.05 0.15 0"/>
+    <origin rpy="0 0 0" xyz="-0.15 0.15 0"/>
     <child link="link_right_wheel"/>
     <parent link="link_chassis"/>
@@ -129,9 +148,9 @@
     <inertial>
       <mass value="0.2"/>
-      <origin rpy="0 1.5707 1.5707" xyz="0 0 0"/>
+      <origin rpy="0 1.5707 1.5707" xyz="-0.15 -0.15 0"/>
       <inertia ixx="0.000526666666667" ixy="0" ixz="0" iyy="0.000526666666667" iyz="0" izz="0.001"/>
     </inertial>
     <collision name="link_left_wheel_collision">
-      <origin rpy="0 1.5707 1.5707" xyz="0 0 0"/>
+      <origin rpy="0 1.5707 1.5707" xyz="-0.15 -0.15 0"/>
       <geometry>
         <cylinder length="0.04" radius="0.1"/>
@@ -139,14 +158,12 @@
     </collision>
     <visual name="link_left_wheel_visual">
-      <!-- <origin rpy="0 1.5707 1.5707" xyz="0 0 0"/> -->
-      <origin rpy="0 1.5707 1.5707" xyz="-0.1 -0.15 0"/>
-      <geometry>
-        <cylinder length="0.06" radius="0.1"/>
-        <!-- <cylinder length="0.04" radius="0.1"/> -->
+      <origin rpy="0 1.5707 1.5707" xyz="-0.15 -0.15 0"/>
+      <geometry>
+        <cylinder length="0.06" radius="0.1"/>
       </geometry>
     </visual>
   </link>
   <joint name="joint_left_wheel" type="continuous">
-    <origin rpy="0 0 0" xyz="-0.05 -0.15 0"/>
+    <origin rpy="0 0 0" xyz="-0.15 -0.15 0"/>
     <child link="link_left_wheel"/>
     <parent link="link_chassis"/>
@@ -155,3 +172,57 @@
     <joint_properties damping="1.0" friction="1.0"/>
   </joint>
+  <link name="front_link_right_wheel">
+    <inertial>
+      <mass value="0.2"/>
+      <origin rpy="0 1.5707 1.5707" xyz="0.15 0.15 0"/>
+      <inertia ixx="0.000526666666667" ixy="0" ixz="0" iyy="0.000526666666667" iyz="0" izz="0.001"/>
+    </inertial>
+    <collision name="front_link_right_wheel_collision">
+      <origin rpy="0 1.5707 1.5707" xyz="0.15 0.15 0"/>
+      <geometry>
+        <cylinder length="0.04" radius="0.1"/>
+      </geometry>
+    </collision>
+    <visual name="front_link_right_wheel_visual">
+      <origin rpy="0 1.5707 1.5707" xyz="0.15 0.15 0"/>
+      <geometry>
+        <cylinder length="0.06" radius="0.1"/>
+      </geometry>
+    </visual>
+  </link>
+  <joint name="front_joint_right_wheel" type="continuous">
+    <origin rpy="0 0 0" xyz="0.15 0.15 0"/>
+    <child link="front_link_right_wheel"/>
+    <parent link="link_chassis"/>
+    <axis rpy="0 0 0" xyz="0 1 0"/>
+    <limit effort="10000" velocity="1000"/>
+    <joint_properties damping="1.0" friction="1.0"/>
+  </joint>
+  <link name="front_link_left_wheel">
+    <inertial>
+      <mass value="0.2"/>
+      <origin rpy="0 1.5707 1.5707" xyz="0.15 -0.15 0"/>
+      <inertia ixx="0.000526666666667" ixy="0" ixz="0" iyy="0.000526666666667" iyz="0" izz="0.001"/>
+    </inertial>
+    <collision name="front_link_left_wheel_collision">
+      <origin rpy="0 1.5707 1.5707" xyz="0.15 -0.15 0"/>
+      <geometry>
+        <cylinder length="0.04" radius="0.1"/>
+      </geometry>
+    </collision>
+    <visual name="front_link_left_wheel_visual">
+      <origin rpy="0 1.5707 1.5707" xyz="0.15 -0.15 0"/>
+      <geometry>
+        <cylinder length="0.06" radius="0.1"/>
+      </geometry>
+    </visual>
+  </link>
+  <joint name="front_joint_left_wheel" type="continuous">
+    <origin rpy="0 0 0" xyz="0.15 -0.15 0"/>
+    <child link="front_link_left_wheel"/>
+    <parent link="link_chassis"/>
+    <axis rpy="0 0 0" xyz="0 1 0"/>
+    <limit effort="10000" velocity="1000"/>
+    <joint_properties damping="1.0" friction="1.0"/>
+  </joint>
 </robot>

File: simulation_ws/src/two_wheel_robot/urdf/two_wheel_robot.xacro (robot description, xacro)
@@ -1,232 +1,153 @@
-<?xml version="1.0" ?>
-<robot name="m2wr" xmlns:xacro="http://www.ros.org/wiki/xacro">
-  <material name="black">
-    <color rgba="0.0 0.0 0.0 1.0"/>
-  </material>
-  <material name="blue">
-    <color rgba="0.203125 0.23828125 0.28515625 1.0"/>
-  </material>
-  <material name="green">
-    <color rgba="0.0 0.8 0.0 1.0"/>
-  </material>
-  <material name="grey">
-    <color rgba="0.2 0.2 0.2 1.0"/>
-  </material>
-  <material name="orange">
-    <color rgba="1.0 0.423529411765 0.0392156862745 1.0"/>
-  </material>
-  <material name="brown">
-    <color rgba="0.870588235294 0.811764705882 0.764705882353 1.0"/>
-  </material>
-  <material name="red">
-    <color rgba="0.80078125 0.12890625 0.1328125 1.0"/>
-  </material>
-  <material name="white">
-    <color rgba="1.0 1.0 1.0 1.0"/>
-  </material>
-  <gazebo reference="link_chassis">
-    <material>Gazebo/Orange</material>
+<?xml version="1.0"?>
+<robot name="two_wheel_robot" xmlns:xacro="http://ros.org/wki/xacro">
+    <material name="black">
+        <color rgba="0.0 0.0 0.0 1.0"/>
+    </material>
+    <material name="blue">
+        <color rgba="0.203125 0.23828125 0.28515625 1.0"/>
+    </material>
+    <material name="green">
+        <color rgba="0.0 0.8 0.0 1.0"/>
+    </material>
+    <material name="grey">
+        <color rgba="0.2 0.2 0.2 1.0"/>
+    </material>
+    <material name="orange">
+        <color rgba="1.0 0.423529411765 0.0392156862745 1.0"/>
+    </material>
+    <material name="brown">
+        <color rgba="0.870588235294 0.811764705882 0.764705882353 1.0"/>
+    </material>
+    <material name="red">
+        <color rgba="0.80078125 0.12890625 0.1328125 1.0"/>
+    </material>
+    <material name="white">
+        <color rgba="1.0 1.0 1.0 1.0"/>
+    </material>
+    <gazebo reference="link_chasis">
+        <material>Gazebo/Orange</material>
+    </gazebo>
+    <gazebo reference="link_left_wheel">
+        <material>Gazebo/Blue</material>
+    </gazebo>
+    <gazebo reference="link_right_wheel">
+        <material>Gazebo/Blue</material>
+    </gazebo>
+    <gazebo>
+        <plugin filename="libgazebo_ros_diff_drive.so" name="differential_drive_controller">
+            <legacyMode>false</legacyMode>
+            <alwaysOn>true</alwaysOn>
+            <updateRate>20</updateRate>
+            <leftJoint>joint_left_wheel</leftJoint>
+            <rightJoint>joint_right_wheel</rightJoint>
+            <wheelSeparation>0.2</wheelSeparation>
+            <wheelDiameter>0.2</wheelDiameter>
+            <torque>0.1</torque>                                    <!-- Can Play with this value -->
+            <commandTopic>cmd_vel</commandTopic>
+            <odometryTopic>odom</odometryTopic>
+            <odometryFrame>odom</odometryFrame>
+            <robotBaseFrame>link_chassis</robotBaseFrame>
+        </plugin>
   </gazebo>
-  <gazebo reference="link_left_wheel">
-    <material>Gazebo/Blue</material>
-  </gazebo>
-  <gazebo reference="link_right_wheel">
-    <material>Gazebo/Blue</material>
-  </gazebo>
-  <gazebo>
-    <plugin filename="libgazebo_ros_diff_drive.so" name="differential_drive_controller">
-      <legacyMode>false</legacyMode>
-      <alwaysOn>true</alwaysOn>
-      <updateRate>20</updateRate>
-      <leftJoint>joint_left_wheel</leftJoint>
-      <rightJoint>joint_right_wheel</rightJoint>
-      <wheelSeparation>0.2</wheelSeparation>
-      <wheelDiameter>0.2</wheelDiameter>
-      <torque>0.1</torque>
-      <commandTopic>cmd_vel</commandTopic>
-      <odometryTopic>odom</odometryTopic>
-      <odometryFrame>odom</odometryFrame>
-      <robotBaseFrame>link_chassis</robotBaseFrame>
-    </plugin>
-  </gazebo>
-  <link name="link_chassis">
-    <!-- pose and inertial -->
-    <pose>0 0 0.1 0 0 0</pose>
-    <inertial>
-      <mass value="5"/>
-      <origin rpy="0 0 0" xyz="0 0 0.1"/>
-      <inertia ixx="0.0395416666667" ixy="0" ixz="0" iyy="0.106208333333" iyz="0" izz="0.106208333333"/>
-    </inertial>
+    <link name="link_chasis">
+        <!-- pose and inertial -->
+        <pose>0 0 00.1 0 0 0</pose>
+        <inertial>
+            <mass value="5"/>
+            <origin rpy="0 0 0" xyz="0 0 0.5"/>
+            <inertia ixx="0.03954166667" ixy="0" ixz="0" iyy="0.106208333333" iyz="0" izz="0.106208333333"/>
+        </inertial>
     <!-- body -->
-    <collision name="collision_chassis">
-      <geometry>
-        <box size="0.5 0.3 0.07"/>
-      </geometry>
+    <collision name="collision_chasis">
+        <geometry>
+            <box size="0.5 0.3 0.07"/>
+        </geometry>
     </collision>
     <visual>
-      <origin rpy="0 0 0" xyz="0 0 0"/>
-      <geometry>
-        <!-- <box size="0.5 0.3 0.07"/> -->
-        <box size="1.0 0.6 0.07"/>
-      </geometry>
-      <material name="blue"/>
+        <origin rpy="0 0 0" xyz=" 0 0 0" />
+        <geometry>
+            <!-- <box size="0.5 0.3 0.7"/> -->
+            <box size="0.6 0.3 0.07"/>
+        </geometry>
+        <material name="blue"/>
     </visual>
-    <!-- caster front -->
+    <!-- caster front: third point for wheels so robot does not fall over-->
     <collision name="caster_front_collision">
-      <origin rpy=" 0 0 0" xyz="0.35 0 -0.05"/>
-      <geometry>
-        <sphere radius="0.05"/>
-      </geometry>
-      <surface>
-        <friction>
-          <ode>
-            <mu>0</mu>
-            <mu2>0</mu2>
-            <slip1>1.0</slip1>
-            <slip2>1.0</slip2>
-          </ode>
-        </friction>
-      </surface>
+        <origin rpy="0 0 0" xyz="0.35 0 -0.05"/>
+        <geometry>
+            <sphere radius="0.05"/>
+        </geometry>
+        <surface>
+            <friction>
+                <ode>
+                    <mu>0</mu>
+                    <mu2>0</mu2>
+                    <slip1>1.0</slip1>
+                    <slip2>1.0</slip2>
+                </ode>
+            </friction>
+        </surface>
     </collision>
     <visual name="caster_front_visual">
-      <!-- <origin rpy=" 0 0 0" xyz="0.2 0 -0.05"/> -->
-      <origin rpy=" 0 0 0" xyz="0.2 0 -0.03"/>
-      <geometry>
-        <sphere radius="0.05"/>
-      </geometry>
+        <origin rpy="0 0 0" xyz="0.2 0 -0.05"/>
+        <geometry>
+            <sphere radius="0.05"/>
+            <!-- <cylinder radius = "0.1" radius="0.05"/> -->
+        </geometry>
     </visual>
-  </link>
-  <link name="link_right_wheel">
-    <inertial>
-      <mass value="0.2"/>
-      <!-- <origin rpy="0 1.5707 1.5707" xyz="0 0 0"/> -->
-      <origin rpy="0 1.5707 1.5707" xyz="-0.15 0.15 0"/>
-      <inertia ixx="0.000526666666667" ixy="0" ixz="0" iyy="0.000526666666667" iyz="0" izz="0.001"/>
-    </inertial>
-    <collision name="link_right_wheel_collision">
-      <!-- <origin rpy="0 1.5707 1.5707" xyz="0 0 0"/> -->
-      <origin rpy="0 1.5707 1.5707" xyz="-0.15 0.15 0"/>
-      <geometry>
-        <cylinder length="0.04" radius="0.1"/>
-      </geometry>
-    </collision>
-    <visual name="link_right_wheel_visual">
-      <!-- <origin rpy="0 1.5707 1.5707" xyz="0 0 0"/> -->
-      <!-- <origin rpy="0 1.5707 1.5707" xyz="-0.1 0.15 0"/> -->
-      <origin rpy="0 1.5707 1.5707" xyz="-0.15 0.15 0"/>
-      <geometry>
-        <cylinder length="0.06" radius="0.1"/>
-        <!-- <cylinder length="0.04" radius="0.1"/> -->
-      </geometry>
-    </visual>
-  </link>
-  <joint name="joint_right_wheel" type="continuous">
-    <origin rpy="0 0 0" xyz="-0.15 0.15 0"/>
-    <!-- <origin rpy="0 0 0" xyz="-0.25 0.15 0"/> -->
-    <child link="link_right_wheel"/>
-    <parent link="link_chassis"/>
-    <axis rpy="0 0 0" xyz="0 1 0"/>
-    <limit effort="10000" velocity="1000"/>
-    <joint_properties damping="1.0" friction="1.0"/>
-  </joint>
-  <link name="link_left_wheel">
-    <inertial>
-      <mass value="0.2"/>
-      <!-- <origin rpy="0 1.5707 1.5707" xyz="0 0 0"/> -->
-      <origin rpy="0 1.5707 1.5707" xyz="-0.15 -0.15 0"/>
-      <inertia ixx="0.000526666666667" ixy="0" ixz="0" iyy="0.000526666666667" iyz="0" izz="0.001"/>
-    </inertial>
-    <collision name="link_left_wheel_collision">
-      <!-- <origin rpy="0 1.5707 1.5707" xyz="0 0 0"/> -->
-      <origin rpy="0 1.5707 1.5707" xyz="-0.15 -0.15 0"/>
-      <geometry>
-        <cylinder length="0.04" radius="0.1"/>
-      </geometry>
-    </collision>
-    <visual name="link_left_wheel_visual">
-      <!-- <origin rpy="0 1.5707 1.5707" xyz="0 0 0"/> -->
-      <!-- <origin rpy="0 1.5707 1.5707" xyz="-0.1 -0.15 0"/> -->
-      <origin rpy="0 1.5707 1.5707" xyz="-0.15 -0.15 0"/>
-      <geometry>
-        <cylinder length="0.06" radius="0.1"/>
-        <!-- <cylinder length="0.04" radius="0.1"/> -->
-      </geometry>
-    </visual>
-  </link>
-  <joint name="joint_left_wheel" type="continuous">
-    <!-- <origin rpy="0 0 0" xyz="-0.05 -0.15 0"/> -->
-    <origin rpy="0 0 0" xyz="-0.15 -0.15 0"/>
-    <child link="link_left_wheel"/>
-    <parent link="link_chassis"/>
-    <axis rpy="0 0 0" xyz="0 1 0"/>
-    <limit effort="10000" velocity="1000"/>
-    <joint_properties damping="1.0" friction="1.0"/>
-  </joint>
-<!-- </robot> -->
-  <link name="front_link_right_wheel">
-    <inertial>
-      <mass value="0.2"/>
-      <!-- <origin rpy="0 1.5707 1.5707" xyz="0 0 0"/> -->
-      <origin rpy="0 1.5707 1.5707" xyz="0.15 0.15 0"/>
-      <inertia ixx="0.000526666666667" ixy="0" ixz="0" iyy="0.000526666666667" iyz="0" izz="0.001"/>
-    </inertial>
-    <collision name="front_link_right_wheel_collision">
-      <!-- <origin rpy="0 1.5707 1.5707" xyz="0 0 0"/> -->
-      <origin rpy="0 1.5707 1.5707" xyz="0.15 0.15 0"/>
-      <geometry>
-        <cylinder length="0.04" radius="0.1"/>
-      </geometry>
-    </collision>
-    <visual name="front_link_right_wheel_visual">
-      <!-- <origin rpy="0 1.5707 1.5707" xyz="0 0 0"/> -->
-      <!-- <origin rpy="0 1.5707 1.5707" xyz="-0.1 0.15 0"/> -->
-      <origin rpy="0 1.5707 1.5707" xyz="0.15 0.15 0"/>
-      <geometry>
-        <cylinder length="0.06" radius="0.1"/>
-        <!-- <cylinder length="0.04" radius="0.1"/> -->
-      </geometry>
-    </visual>
-  </link>
-  <joint name="front_joint_right_wheel" type="continuous">
-    <origin rpy="0 0 0" xyz="0.15 0.15 0"/>
-    <!-- <origin rpy="0 0 0" xyz="-0.25 0.15 0"/> -->
-    <child link="front_link_right_wheel"/>
-    <parent link="link_chassis"/>
-    <axis rpy="0 0 0" xyz="0 1 0"/>
-    <limit effort="10000" velocity="1000"/>
-    <joint_properties damping="1.0" friction="1.0"/>
-  </joint>
-  <link name="front_link_left_wheel">
-    <inertial>
-      <mass value="0.2"/>
-      <!-- <origin rpy="0 1.5707 1.5707" xyz="0 0 0"/> -->
-      <origin rpy="0 1.5707 1.5707" xyz="0.15 -0.15 0"/>
-      <inertia ixx="0.000526666666667" ixy="0" ixz="0" iyy="0.000526666666667" iyz="0" izz="0.001"/>
-    </inertial>
-    <collision name="front_link_left_wheel_collision">
-      <!-- <origin rpy="0 1.5707 1.5707" xyz="0 0 0"/> -->
-      <origin rpy="0 1.5707 1.5707" xyz="0.15 -0.15 0"/>
-      <geometry>
-        <cylinder length="0.04" radius="0.1"/>
-      </geometry>
-    </collision>
-    <visual name="front_link_left_wheel_visual">
-      <!-- <origin rpy="0 1.5707 1.5707" xyz="0 0 0"/> -->
-      <!-- <origin rpy="0 1.5707 1.5707" xyz="-0.1 -0.15 0"/> -->
-      <origin rpy="0 1.5707 1.5707" xyz="0.15 -0.15 0"/>
-      <geometry>
-        <cylinder length="0.06" radius="0.1"/>
-        <!-- <cylinder length="0.04" radius="0.1"/> -->
-      </geometry>
-    </visual>
-  </link>
-  <joint name="front_joint_left_wheel" type="continuous">
-    <!-- <origin rpy="0 0 0" xyz="-0.05 -0.15 0"/> -->
-    <origin rpy="0 0 0" xyz="0.15 -0.15 0"/>
-    <child link="front_link_left_wheel"/>
-    <parent link="link_chassis"/>
-    <axis rpy="0 0 0" xyz="0 1 0"/>
-    <limit effort="10000" velocity="1000"/>
-    <joint_properties damping="1.0" friction="1.0"/>
-  </joint>
+    </link>
+    <link name="link_right_wheel">
+        <inertial>
+            <mass value="0.2"/>
+            <origin rpy="0 1.5707 1.5707" xyz="0 0 0"/>
+            <inertia ixx="0.000526666666667" ixy="0" ixz="0" iyy="0.000526666666667" iyz="0" izz="0.001"/>
+        </inertial>
+        <collision name="link_right_wheel_collision">
+            <origin rpy="0 1.5707 1.5707" xyz="0 0 0"/>
+            <geometry>
+                <cylinder length="0.04" radius="0.1"/>
+            </geometry>
+        </collision>
+        <visual name="link_right_wheel_visual">
+            <origin rpy="0 1.5707 1.5707" xyz="0 0 0"/>
+            <geometry>
+                <cylinder length="0.04" radius="0.1"/>
+            </geometry>
+        </visual>
+    </link>
+    <joint name="joint_right_wheel" type="continuous">
+        <origin rpy="0 0 0" xyz="-0.05 0.15 0"/>
+        <child link="link_right_wheel"/>
+        <parent link="link_chasis"/>
+        <axis rpy="0 0 0" xyz="0 1 0"/>
+        <limit effort="10000" velocity="1000"/>
+        <joint_properties damping="1.0" friction="1.0"/>
+    </joint>
+    <link name="link_left_wheel">
+        <inertial>
+            <mass value="0.2"/>
+            <origin rpy="0 1.5707 1.5707" xyz="0 0 0"/>
+            <inertia ixx="0.000526666666667" ixy="0" ixz="0" iyy="0.000526666666667" iyz="0" izz="0.001"/>
+        </inertial>
+        <collision name="link_left_wheel_collision">
+            <origin rpy="0 1.5707 1.5707" xyz="0 0 0"/>
+            <geometry>
+                <cylinder length="0.04" radius="0.1"/>
+            </geometry>
+        </collision>
+        <visual name="link_left_wheel_visual">
+            <origin rpy="0 1.5707 1.5707" xyz="0 0 0"/>
+            <geometry>
+                <cylinder length="0.04" radius="0.1"/>
+            </geometry>
+        </visual>
+    </link>
+    <joint name="joint_left_wheel" type="continuous">
+        <origin rpy="0 0 0" xyz="-0.05 -0.15 0"/>
+        <child link="link_left_wheel"/>
+        <parent link="link_chasis"/>
+        <axis rpy="0 0 0" xyz="0 1 0"/>
+        <limit effort="10000" velocity="1000"/>
+        <joint_properties damping="1.0" friction="1.0"/>
+    </joint>
 </robot>
