Commit message: fix un-froglike driving on 4 wheel car

File: simulation_ws/src/two_wheel_robot/urdf/4_two_wheel_robot.xacro (robot description, xacro)
@@ -1,4 +1,4 @@
 <?xml version="1.0" ?>
-<robot name="m2wr" xmlns:xacro="http://www.ros.org/wiki/xacro">
+<robot name="two_wheel_robot" xmlns:xacro="http://www.ros.org/wiki/xacro">
   <material name="black">
     <color rgba="0.0 0.0 0.0 1.0"/>
@@ -41,7 +41,9 @@
       <leftJoint>joint_left_wheel</leftJoint>
       <rightJoint>joint_right_wheel</rightJoint>
+      <rightJoint>front_joint_right_wheel</rightJoint>
+      <leftJoint>front_joint_left_wheel</leftJoint>
       <wheelSeparation>0.2</wheelSeparation>
       <wheelDiameter>0.2</wheelDiameter>
-      <torque>0.1</torque>
+      <torque>0.5</torque>
       <commandTopic>cmd_vel</commandTopic>
       <odometryTopic>odom</odometryTopic>
@@ -61,5 +63,5 @@
     <collision name="collision_chassis">
       <geometry>
-        <box size="0.5 0.3 0.07"/>
+        <box size="1.0 0.6 0.07"/>
       </geometry>
     </collision>
@@ -72,5 +74,5 @@
     </visual>
     <!-- caster front -->
-    <collision name="caster_front_collision">
+<!--     <collision name="caster_front_collision">
       <origin rpy=" 0 0 0" xyz="0.35 0 -0.05"/>
       <geometry>
@@ -94,6 +96,7 @@
       </geometry>
     </visual>
+ -->
     <!-- caster rear -->
-    <collision name="caster_front_collision">
+<!--     <collision name="caster_front_collision">
     <origin rpy=" 0 0 0" xyz="-0.35 0 -0.05"/>
       <geometry>
@@ -117,9 +120,10 @@
       </geometry>
     </visual>
+ -->
   </link>
   <link name="link_right_wheel">
     <inertial>
       <mass value="0.2"/>
-      <origin rpy="0 1.5707 1.5707" xyz="0.15 0.15 0"/>
+      <origin rpy="0 1.5707 1.5707" xyz="-0.15 0.15 0"/>
       <inertia ixx="0.000526666666667" ixy="0" ixz="0" iyy="0.000526666666667" iyz="0" izz="0.001"/>
     </inertial>
@@ -138,4 +142,5 @@
   </link>
   <joint name="joint_right_wheel" type="continuous">
+  <!-- <joint name="joint_right_wheel" type="fixed"> -->
     <origin rpy="0 0 0" xyz="-0.15 0.15 0"/>
     <child link="link_right_wheel"/>
@@ -165,4 +170,5 @@
   </link>
   <joint name="joint_left_wheel" type="continuous">
+  <!-- <joint name="joint_left_wheel" type="fixed"> -->
     <origin rpy="0 0 0" xyz="-0.15 -0.15 0"/>
     <child link="link_left_wheel"/>
@@ -191,5 +197,6 @@
     </visual>
   </link>
-  <joint name="front_joint_right_wheel" type="continuous">
+  <!-- <joint name="front_joint_right_wheel" type="continuous"> -->
+  <joint name="front_joint_right_wheel" type="fixed">
     <origin rpy="0 0 0" xyz="0.15 0.15 0"/>
     <child link="front_link_right_wheel"/>
@@ -218,5 +225,6 @@
     </visual>
   </link>
-  <joint name="front_joint_left_wheel" type="continuous">
+  <!-- <joint name="front_joint_left_wheel" type="continuous"> -->
+  <joint name="front_joint_left_wheel" type="fixed">
     <origin rpy="0 0 0" xyz="0.15 -0.15 0"/>
     <child link="front_link_left_wheel"/>

File: simulation_ws/src/two_wheel_robot/urdf/4_two_wheel_robot_revA.xacro (robot description, xacro)
@@ -151,5 +151,6 @@
   <joint name="front_joint_right_wheel" type="continuous">
   <!-- <joint name="front_joint_right_wheel" type="fixed"> -->
-    <origin rpy="0 0 0" xyz="0.15 0.15 0"/>
+    <!-- <origin rpy="0 0 0" xyz="0.15 0.15 0"/> -->
+    <origin rpy="0 0 0" xyz="0.45 0.15 0"/>
     <child link="front_link_right_wheel"/>
     <parent link="link_chassis"/>
@@ -179,5 +180,6 @@
   <joint name="front_joint_left_wheel" type="continuous">
   <!-- <joint name="front_joint_left_wheel" type="fixed"> -->
-    <origin rpy="0 0 0" xyz="0.15 -0.15 0"/>
+    <!-- <origin rpy="0 0 0" xyz="0.15 -0.15 0"/> -->
+    <origin rpy="0 0 0" xyz="0.45 -0.15 0"/>
     <child link="front_link_left_wheel"/>
     <parent link="link_chassis"/>
